File: RS485 Test.kicad_pcb (KiCad board)
At the start: 4 copper layers, 69.6 x 39.4 mm, 49 parts, among them J1 USB_C_Receptacle_USB2.0, J2 Conn_ARM_JTAG_SWD_10, J3 Conn_02x03_Odd_Even, J4 Floor Connector, J5 IDC, J6 Conn_01x05_Female, SW1 SW_SPST, U1 AP1117-33, U2 STM32F103C8Tx, U3 MAX3078E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

Commit message: Fixing DRC issues
Connections:
- J1 pad : Net-(F1-Pad2) -> (no net)
Routing:
- net Net-(F1-Pad2): track 14.5 -> 7.75 mm, vias 0 -> 5
- added copper zone on In1.Cu, net Net-(F1-Pad2)
